File: Controller.brd (EAGLE design)
At the start: 125 x 65 mm, 35 parts, among them SW1 MULTICOLOR_BUTTON, SW10 MY_LBR_SPSTSWITCH, SW2 MULTICOLOR_BUTTON, SW3 MULTICOLOR_BUTTON, SW4 MULTICOLOR_BUTTON, SW5 MULTICOLOR_BUTTON, SW6 MULTICOLOR_BUTTON, SW7 MULTICOLOR_BUTTON, SW8 MULTICOLOR_BUTTON, SW9 MY_LBR_SPSTSWITCH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

Commit message: Redoing the board
Parts:
- removed R20, R21, R22, R23: 1k, rcl:R1206
- removed R24, R25: 10k, rcl:R1206
- removed R26: 100k, rcl:R1206
- removed SW10, SW9: MY_LBR_SPSTSWITCH, Controller:MY_LBR_2HOLES
- removed U$2, U$3: BUMPER_BUMPER, Controller:BUMPER_BUMPER
- added C1, C2, C9: 0.1u, rcl:C1206
- added C4, C6: 22p, rcl:C1206
- added C7: 10u, rcl:C1206
- added C8: 10U, rcl:C1206
- added Q1: (no value), crystal:HC49/S
- added R1, R2, R3, R4: 100k, rcl:R1206
- added U3: DRV5053VAQLPGM, Controller:LPG3
- added U4: LM1086IT-3.3/NOPB, Controller:T03B
- C3: value 10uF -> 0.1u
- C5: value 22pF -> 0.1u
- U2: value MCP6002T-I/SNSOIC8-N_MC-M -> DRV5053VAQLPGM; device Controller:SOIC8-N_MC-M -> Controller:LPG3
- moved U2 216.7 mm to (-9.10, -189.8)
- moved C3 184.5 mm to (-11.0, -152.6), turned to 0 degrees
- moved U$4 177.4 mm to (92.8, 61.4), turned to 180 degrees
- moved U$6 173.8 mm to (32.6, 62.3), turned to 180 degrees
- moved U1 126.9 mm to (70.7, 24.5)
- moved C5 114.5 mm to (-11.0, -183.6)
- moved R15 29.3 mm to (47.7, 33.6), turned to 0 degrees
- moved SW1 17.0 mm to (20.0, 33.0)
- moved SW3 17.0 mm to (8.00, 45.0)
- moved SW5 17.0 mm to (93.0, 45.0), turned to 180 degrees
- moved SW8 17.0 mm to (105.0, 57.0), turned to 180 degrees
- moved XB2 8.82 mm to (62.5, 45.0), turned to 0 degrees
- turned SW7 to 180 degrees
Connections:
- removed net LEFT_BUTTON_OUTPUT: C5.1, R26.1, U2.3
- removed net LEFT_OUTPUT: U2.1, U2.2
- removed net N$13: R21.1, R22.2, U$3.P$1
- removed net N$18: R22.1, R23.2, SW9.P$1
- removed net N$19: R23.1, R24.2, SW10.P$1
- removed net N$2: R20.1, R21.2, U$2.P$1
- removed net N$20: R24.1, R25.2
- removed net N$21: R26.2, SW10.P$2, SW9.P$2, U$2.P$2, U$3.P$2
- removed net N$24: U1.24
- removed net N$25: U1.23
- removed net N$5: S1.B1A, S2.B1A, U$4.P$1, U$6.P$1
- removed net RIGHT_BUTTON_OUTPUT: U2.5
- removed net RIGHT_OUTPUT: U2.6, U2.7
- new net $NC2: S2.B2A, SW2.4, SW6.4
- new net N$C1: C1.1, R1.1, S1.B2A, SW1.4, SW5.4
- new net N$C2: C2.1, R2.1
- new net N$C3: C3.1, R3.1, SW3.4, SW7.4, U$4.P$2
- new net N$C4: C5.1, R4.1, SW4.4, SW8.4, U$6.P$2
- new net R1: SW1.2, SW2.2, SW3.2, SW4.2, U1.17
- new net R2: SW5.2, SW6.2, SW7.2, SW8.2, U1.16
- new net R3: S1.B1A, S2.B1A, U$4.P$1, U$6.P$1, U1.15
- new net TRIGGER_LEFT: U1.24, U2.3
- new net TRIGGER_RIGHT: U1.23, U3.3
- net +3V3: now also C7.1, C9.1, U4.2
- net +5V: now also C8.1, U2.1, U3.1, U4.3; no longer C3.1, R20.2, U2.8
- net C1: now also R1.2, U1.4; no longer S1.B2A, SW1.4, SW5.4
- net C2: now also R2.2, U1.5; no longer S2.B2A, SW2.4, SW6.4
- net C3: now also R3.2, U1.11; no longer SW3.4, SW7.4, U$4.P$4
- net C4: now also R4.2, U1.14; no longer SW4.4, SW8.4, U$6.P$4
- net GND: now also C1.2, C2.2, C4.2, C6.2, C7.2, C8.2, C9.2, U2.2, U3.2, U4.1; no longer R25.1, U$2.P$3, U$2.P$4, U$3.P$3, U$3.P$4, U2.4
- net N$3: now also C4.1, Q1.1, U1.9; no longer SW1.2, SW2.2, SW3.2, SW4.2
- net N$4: now also C6.1, Q1.2, U1.10; no longer SW5.2, SW6.2, SW7.2, SW8.2
Routing:
- net N$C4: track 0.00 -> 138.7 mm, vias 0 -> 4
- net $NC2: track 0.00 -> 114.0 mm, vias 0 -> 1
- net R1: track 0.00 -> 106.4 mm
- net R2: track 0.00 -> 73.0 mm
- net +5V: track 59.5 -> 0.00 mm, vias 8 -> 6
- net +3V3: track 68.1 -> 10.8 mm, vias 4 -> 0
- net N$17: track 54.3 -> 2.52 mm, vias 1 -> 0
- net X_LEFT: track 50.2 -> 0.00 mm, vias 2 -> 0
- net N$14: track 53.5 -> 3.82 mm, vias 1 -> 0
- net RIGHT_OUTPUT: track 47.0 -> 0.00 mm, vias 2 -> 0
- net R3: track 0.00 -> 44.3 mm, vias 0 -> 1
- net Y_LEFT: track 63.3 -> 23.9 mm
- net RIGHT_BUTTON_OUTPUT: track 35.5 -> 0.00 mm
- net N$C3: track 0.00 -> 28.8 mm
- net N$C1: track 0.00 -> 27.7 mm
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- added copper zone on layer 16, net +5V
- removed copper zone on layer 1, net GND

Commit message: Added Board
Parts:
- moved C9 272.1 mm to (53.6, 47.6), flipped to the bottom, turned to 270 degrees
- moved U3 265.8 mm to (106.5, 44.9), flipped to the bottom, turned to 180 degrees
- moved C8 261.4 mm to (64.7, 39.7), flipped to the bottom, turned to 270 degrees
- moved C5 247.6 mm to (82.7, 45.6), turned to 180 degrees
- moved R4 244.2 mm to (82.8, 48.1), turned to 180 degrees
- moved U2 236.1 mm to (21.0, 44.3), flipped to the bottom, turned to 180 degrees
- moved R3 220.0 mm to (94.1, 34.5), turned to 180 degrees
- moved C4 217.9 mm to (58.4, 41.6)
- moved C3 212.6 mm to (94.2, 32.2), turned to 180 degrees
- moved C7 211.0 mm to (11.2, 5.54), turned to 180 degrees
- moved C6 210.6 mm to (58.7, 27.5)
- moved U4 207.8 mm to (15.3, 8.95), flipped to the bottom, turned to 180 degrees
- moved R2 205.3 mm to (94.2, 29.9), turned to 180 degrees
- moved C2 198.0 mm to (94.3, 27.5), turned to 180 degrees
- moved R1 173.4 mm to (30.7, 34.3)
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Routing:
- net +3V3: track 10.8 -> 109.1 mm, vias 0 -> 1
- net GND: track 23.4 -> 115.5 mm, vias 0 -> 5
- net +5V: track 0.00 -> 91.4 mm, vias 6 -> 0
- net R3: track 44.3 -> 129.8 mm, vias 1 -> 2
- net C1: track 0.00 -> 78.4 mm, vias 0 -> 1
- net X_LEFT: track 0.00 -> 76.4 mm, vias 0 -> 1
- net N$C1: track 27.7 -> 100.4 mm, vias 0 -> 2
- net TRIGGER_LEFT: track 0.00 -> 70.2 mm
- net N$C3: track 28.8 -> 97.1 mm
- net C2: track 0.00 -> 50.0 mm, vias 0 -> 3
- net $NC2: track 114.0 -> 161.8 mm, vias 1 -> 0
- net TRIGGER_RIGHT: track 0.00 -> 46.2 mm
- net C4: track 0.00 -> 44.8 mm, vias 0 -> 3
- net Y_LEFT: track 23.9 -> 67.8 mm
- net C3: track 0.00 -> 32.6 mm, vias 0 -> 1
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- added copper zone on layer 2, net +5V
- added copper zone on layer 1, net GND
- added copper zone on layer 15, net GND
- removed copper zone on layer 1, net +5V
- removed copper zone on layer 16, net +5V
- removed copper zone on layer 16, net GND
Other:
- outline, holes or cut-outs redrawn
