File: Electrical/Board Files/ControllerPower.kicad_sch (KiCad schematic)
At the start: 41 parts

Commit message: added switch
Parts:
- added SW?: SW_DIP_x01, symbol Switch:SW_DIP_x01
Connections:
- net VCC: now also SW?.2; no longer J?.2 (Pin_2)
- new net: J?.2 (Pin_2), SW?.1
Other:
- moved on the sheet: J?
Changed lines of the file:
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@@
   (junction (at 226.822 124.587) (diameter 0) (color 0 0 0 0)
   )
+  (junction (at 87.376 59.055) (diameter 0) (color 0 0 0 0)
+  )
   (junction (at 111.379 57.023) (diameter 0) (color 0 0 0 0)
   )
@@
   (junction (at 226.822 133.096) (diameter 0) (color 0 0 0 0)
   )
-  (junction (at 87.376 61.214) (diameter 0) (color 0 0 0 0)
-  )
   (junction (at 107.696 61.214) (diameter 0) (color 0 0 0 0)
   )
@@
     (stroke (width 0) (type default) (color 0 0 0 0))
   )
+  (wire (pts (xy 87.376 59.055) (xy 87.376 61.214))
+    (stroke (width 0) (type default) (color 0 0 0 0))
+  )
   (wire (pts (xy 134.366 149.352) (xy 134.366 147.066))
     (stroke (width 0) (type default) (color 0 0 0 0))
@@
     (stroke (width 0) (type default) (color 0 0 0 0))
   )
+  (wire (pts (xy 52.578 59.055) (xy 52.578 61.214))
+    (stroke (width 0) (type default) (color 0 0 0 0))
+  )
   (wire (pts (xy 201.549 124.587) (xy 210.82 124.587))
     (stroke (width 0) (type default) (color 0 0 0 0))
@@
     (stroke (width 0) (type default) (color 0 0 0 0))
   )
+  (wire (pts (xy 52.578 61.214) (xy 49.53 61.214))
+    (stroke (width 0) (type default) (color 0 0 0 0))
+  )
   (wire (pts (xy 134.366 134.747) (xy 143.51 134.747))
     (stroke (width 0) (type default) (color 0 0 0 0))
@@
     (stroke (width 0) (type default) (color 0 0 0 0))
   )
-  (wire (pts (xy 94.361 79.629) (xy 115.189 79.629))
-    (stroke (width 0) (type default) (color 0 0 0 0))
-  )
-  (wire (pts (xy 78.232 63.754) (xy 94.361 63.754))
+  (wire (pts (xy 84.582 79.629) (xy 115.189 79.629))
+    (stroke (width 0) (type default) (color 0 0 0 0))
+  )
+  (wire (pts (xy 49.53 63.754) (xy 84.582 63.754))
     (stroke (width 0) (type default) (color 0 0 0 0))
   )
@@
     (stroke (width 0) (type default) (color 0 0 0 0))
   )
-  (wire (pts (xy 87.376 54.483) (xy 87.376 61.214))
+  (wire (pts (xy 87.376 54.483) (xy 87.376 59.055))
     (stroke (width 0) (type default) (color 0 0 0 0))
   )
@@
     (stroke (width 0) (type default) (color 0 0 0 0))
   )
+  (wire (pts (xy 84.582 79.629) (xy 84.582 63.754))
+    (stroke (width 0) (type default) (color 0 0 0 0))
+  )
   (wire (pts (xy 162.941 74.549) (xy 164.846 74.549))
     (stroke (width 0) (type default) (color 0 0 0 0))
@@
     (stroke (width 0) (type default) (color 0 0 0 0))
   )
-  (wire (pts (xy 78.232 61.214) (xy 87.376 61.214))
-    (stroke (width 0) (type default) (color 0 0 0 0))
-  )
   (wire (pts (xy 111.379 51.562) (xy 111.379 57.023))
     (stroke (width 0) (type default) (color 0 0 0 0))
@@
     (stroke (width 0) (type default) (color 0 0 0 0))
   )
+  (wire (pts (xy 67.818 59.055) (xy 87.376 59.055))
+    (stroke (width 0) (type default) (color 0 0 0 0))
+  )
   (wire (pts (xy 165.481 49.784) (xy 165.481 51.054))
     (stroke (width 0) (type default) (color 0 0 0 0))
@@
   )
   (wire (pts (xy 168.402 134.239) (xy 177.8 134.239))
-    (stroke (width 0) (type default) (color 0 0 0 0))
-  )
-  (wire (pts (xy 94.361 63.754) (xy 94.361 79.629))
     (stroke (width 0) (type default) (color 0 0 0 0))
   )
@@
     (pin "2")
   )
+  (symbol (lib_id "Switch:SW_DIP_x01") (at 60.198 59.055 0) (unit 1)
+    (in_bom yes) (on_board yes)
+    (property "Reference" "SW?" (id 0) (at 53.975 57.15 0))
+    (property "Value" "SW_DIP_x01" (id 1) (at 70.231 61.595 0)
+      (effects (font (size 1.27 1.27)) hide)
+    )
+    (property "Footprint" "" (id 2) (at 60.198 59.055 0)
+      (effects (font (size 1.27 1.27)) hide)
+    )
+    (property "Datasheet" "~" (id 3) (at 60.198 59.055 0)
+      (effects (font (size 1.27 1.27)) hide)
+    )
+    (pin "1")
+    (pin "2")
+  )
   (symbol (lib_id "power:GND") (at 192.786 68.199 0) (unit 1)
     (in_bom yes) (on_board yes) (fields_autoplaced)
@@
     (pin "1")
   )
-  (symbol (lib_id "Connector:Conn_01x02_Female") (at 73.152 63.754 180) (unit 1)
+  (symbol (lib_id "Connector:Conn_01x02_Female") (at 44.45 63.754 180) (unit 1)
     (in_bom yes) (on_board yes) (fields_autoplaced)
-    (property "Reference" "J?" (id 0) (at 73.787 58.674 0))
-    (property "Value" "Conn_01x02_Female" (id 1) (at 73.787 58.674 0)
-      (effects (font (size 1.27 1.27)) hide)
-    )
-    (property "Footprint" "" (id 2) (at 73.152 63.754 0)
-      (effects (font (size 1.27 1.27)) hide)
-    )
-    (property "Datasheet" "~" (id 3) (at 73.152 63.754 0)
-      (effects (font (size 1.27 1.27)) hide)
-    )
+    (property "Reference" "J?" (id 0) (at 45.085 58.674 0))
+    (property "Value" "Conn_01x02_Female" (id 1) (at 45.085 58.674 0)
+      (effects (font (size 1.27 1.27)) hide)
+    )
+    (property "Footprint" "" (id 2) (at 44.45 63.754 0)
+      (effects (font (size 1.27 1.27)) hide)
+    )
+    (property "Datasheet" "~" (id 3) (at 44.45 63.754 0)
+      (effects (font (size 1.27 1.27)) hide)
+    )

Commit message: Added Xbee libs and bus aliases
Parts:
- gave numbers to parts that had none: 42
Other:
- title: (none) -> Robotics Controller
