File: Electrical/Board Files/Debug.kicad_sch (KiCad schematic)
At the start: 16 parts, among them J2 Conn_01x04_Female, J3 USB_B_Micro, U8 FT231XS

Commit message: Fixing USB pins and added SPI_CS
Parts:
- removed J2: Conn_01x04_Female, symbol Connector:Conn_01x04_Female
- added J2: Conn_01x05_Female, symbol Connector:Conn_01x05_Female
Connections:
- net +3V3: now also J2.1 (Pin_1)
- net GND: now also J2.5 (Pin_5)
- net SWD.CLK: now also J2.3 (Pin_3)
- net SWD.DATA: now also J2.2 (Pin_2)
- net at R22.1: now also J3.2 (D-); no longer J3.3 (D+)
- net at R23.1: now also J3.3 (D+); no longer J3.2 (D-)
- new net SWD.NRST: J2.4 (Pin_4)
Changed lines of the file:
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@@
+    (stroke (width 0) (type default) (color 0 0 0 0))
+  )
+  (bus_entry (at 85.217 104.902) (size -2.54 -2.54)
     (stroke (width 0) (type default) (color 0 0 0 0))
   )
@@
     (stroke (width 0) (type default) (color 0 0 0 0))
   )
-  (wire (pts (xy 69.088 102.362) (xy 69.088 105.537))
+  (wire (pts (xy 69.088 104.902) (xy 69.088 108.204))
     (stroke (width 0) (type default) (color 0 0 0 0))
   )
@@
     (stroke (width 0) (type default) (color 0 0 0 0))
   )
+  (bus (pts (xy 85.217 104.902) (xy 85.217 106.172))
+    (stroke (width 0) (type default) (color 0 0 0 0))
+  )
+  (wire (pts (xy 46.228 102.362) (xy 82.677 102.362))
+    (stroke (width 0) (type default) (color 0 0 0 0))
+  )
   (wire (pts (xy 133.731 93.98) (xy 133.731 95.25))
     (stroke (width 0) (type default) (color 0 0 0 0))
@@
     (stroke (width 0) (type default) (color 0 0 0 0))
   )
-  (wire (pts (xy 46.228 102.362) (xy 69.088 102.362))
+  (wire (pts (xy 46.228 104.902) (xy 69.088 104.902))
     (stroke (width 0) (type default) (color 0 0 0 0))
   )
@@
     (stroke (width 0) (type default) (color 0 0 0 0))
   )
-  (bus (pts (xy 85.217 102.362) (xy 85.217 106.172))
+  (bus (pts (xy 85.217 102.362) (xy 85.217 104.902))
     (stroke (width 0) (type default) (color 0 0 0 0))
   )
@@
   )
   (label "DCD_B" (at 204.851 104.14 0)
+    (effects (font (size 1.27 1.27)) (justify left bottom))
+  )
+  (label "SWD.NRST" (at 52.705 102.362 0)
     (effects (font (size 1.27 1.27)) (justify left bottom))
   )
@@
     (pin "1")
   )
-  (symbol (lib_id "power:GND") (at 69.088 105.537 0) (unit 1)
-    (in_bom yes) (on_board yes) (fields_autoplaced)
-    (property "Reference" "#PWR043" (id 0) (at 69.088 111.887 0)
-      (effects (font (size 1.27 1.27)) hide)
-    )
-    (property "Value" "GND" (id 1) (at 69.088 110.363 0))
-    (property "Footprint" "" (id 2) (at 69.088 105.537 0)
-      (effects (font (size 1.27 1.27)) hide)
-    )
-    (property "Datasheet" "" (id 3) (at 69.088 105.537 0)
+  (symbol (lib_id "power:GND") (at 69.088 108.204 0) (unit 1)
+    (in_bom yes) (on_board yes) (fields_autoplaced)
+    (property "Reference" "#PWR043" (id 0) (at 69.088 114.554 0)
+      (effects (font (size 1.27 1.27)) hide)
+    )
+    (property "Value" "GND" (id 1) (at 69.088 113.03 0))
+    (property "Footprint" "" (id 2) (at 69.088 108.204 0)
+      (effects (font (size 1.27 1.27)) hide)
+    )
+    (property "Datasheet" "" (id 3) (at 69.088 108.204 0)
       (effects (font (size 1.27 1.27)) hide)
     )
@@
     (pin "1")
     (pin "2")
+  )
+  (symbol (lib_id "Connector:Conn_01x05_Female") (at 41.148 99.822 0) (mirror y) (unit 1)
+    (in_bom yes) (on_board yes) (fields_autoplaced)
+    (property "Reference" "J2" (id 0) (at 41.783 88.9 0))
+    (property "Value" "Conn_01x05_Female" (id 1) (at 41.783 91.44 0))
+    (property "Footprint" "" (id 2) (at 41.148 99.822 0)
+      (effects (font (size 1.27 1.27)) hide)
+    )
+    (property "Datasheet" "~" (id 3) (at 41.148 99.822 0)
+      (effects (font (size 1.27 1.27)) hide)
+    )
+    (pin "1")
+    (pin "2")
+    (pin "3")
+    (pin "4")
+    (pin "5")
   )
   (symbol (lib_id "power:+3V3") (at 69.088 90.932 0) (unit 1)
@@
     (pin "1")
   )
-  (symbol (lib_id "Connector:Conn_01x04_Female") (at 41.148 97.282 0) (mirror y) (unit 1)
-    (in_bom yes) (on_board yes) (fields_autoplaced)
-    (property "Reference" "J2" (id 0) (at 41.783 89.154 0))
-    (property "Value" "Conn_01x04_Female" (id 1) (at 41.783 91.694 0))
-    (property "Footprint" "" (id 2) (at 41.148 97.282 0)
-      (effects (font (size 1.27 1.27)) hide)
-    )
-    (property "Datasheet" "~" (id 3) (at 41.148 97.282 0)
-      (effects (font (size 1.27 1.27)) hide)
-    )
-    (pin "1")
-    (pin "2")
-    (pin "3")
-    (pin "4")
-  )
   (symbol (lib_id "Connector:TestPoint") (at 223.901 144.78 270) (unit 1)

Commit message: Adding some device footprints and MPN
Parts:
- C36: MANUFACTURER (none) -> CL10A105KB8NNNC
- D19: footprint (none) -> LED_SMD:LED_0603_1608Metric; MANUFACTURER (none) -> BL-HG036D-AV-TRB
- D20: value ~ -> -; footprint (none) -> Diode_SMD:D_SOD-323; MANUFACTURER (none) -> 1N4148WS
- R22, R23, R24, R25: footprint (none) -> Resistor_SMD:R_0603_1608Metric
- TP15: footprint (none) -> TestPoint:TestPoint_THTPad_2.0x2.0mm_Drill1.0mm
- TP16, TP17, TP18, TP19, TP20: value ~ -> TestPoint; footprint (none) -> TestPoint:TestPoint_THTPad_2.0x2.0mm_Drill1.0mm
Changed lines of the file:
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@@
       (effects (font (size 1.27 1.27)) (justify right))
     )
-    (property "Value" "~" (id 1) (at 223.901 107.2514 90)
+    (property "Value" " - " (id 1) (at 223.901 107.2514 90)
       (effects (font (size 1.27 1.27)) (justify right) hide)
     )
-    (property "Footprint" "" (id 2) (at 221.996 106.045 90)
+    (property "Footprint" "Diode_SMD:D_SOD-323" (id 2) (at 221.996 106.045 90)
       (effects (font (size 1.27 1.27)) hide)
     )
     (property "Datasheet" "~" (id 3) (at 221.996 106.045 90)
+      (effects (font (size 1.27 1.27)) hide)
+    )
+    (property "MANUFACTURER" "1N4148WS" (id 4) (at 221.996 106.045 0)
       (effects (font (size 1.27 1.27)) hide)
     )
@@
       (effects (font (size 1.27 1.27)) (justify left))
     )
-    (property "Value" "~" (id 1) (at 228.981 143.5099 90)
-      (effects (font (size 1.27 1.27)) (justify left))
-    )
-    (property "Footprint" "" (id 2) (at 223.901 147.32 0)
+    (property "Value" "TestPoint" (id 1) (at 228.981 143.5099 90)
+      (effects (font (size 1.27 1.27)) (justify left))
+    )
+    (property "Footprint" "TestPoint:TestPoint_THTPad_2.0x2.0mm_Drill1.0mm" (id 2) (at 223.901 147.32 0)
       (effects (font (size 1.27 1.27)) hide)
     )
@@
       (effects (font (size 1.27 1.27)) (justify left))
     )
-    (property "Footprint" "" (id 2) (at 214.122 98.679 90)
+    (property "Footprint" "Resistor_SMD:R_0603_1608Metric" (id 2) (at 214.122 98.679 90)
       (effects (font (size 1.27 1.27)) hide)
     )
@@
     (property "Reference" "R22" (id 0) (at 141.986 95.885 90))
     (property "Value" "27R" (id 1) (at 146.431 92.71 90))
-    (property "Footprint" "" (id 2) (at 141.986 93.98 0)
+    (property "Footprint" "Resistor_SMD:R_0603_1608Metric" (id 2) (at 141.986 93.98 0)
       (effects (font (size 1.27 1.27)) hide)
     )
@@
       (effects (font (size 1.27 1.27)) (justify left) hide)
     )
-    (property "Footprint" "" (id 2) (at 223.901 144.78 0)
+    (property "Footprint" "TestPoint:TestPoint_THTPad_2.0x2.0mm_Drill1.0mm" (id 2) (at 223.901 144.78 0)
       (effects (font (size 1.27 1.27)) hide)
     )
@@
     (property "Reference" "R23" (id 0) (at 142.621 100.965 90))
     (property "Value" "27R" (id 1) (at 145.796 97.79 90))
-    (property "Footprint" "" (id 2) (at 141.986 99.06 0)
+    (property "Footprint" "Resistor_SMD:R_0603_1608Metric" (id 2) (at 141.986 99.06 0)
       (effects (font (size 1.27 1.27)) hide)
     )
@@
       (effects (font (size 1.27 1.27)) (justify right) hide)
     )
-    (property "Footprint" "" (id 2) (at 213.106 106.045 90)
+    (property "Footprint" "LED_SMD:LED_0603_1608Metric" (id 2) (at 213.106 106.045 90)
       (effects (font (size 1.27 1.27)) hide)
     )
@@
       (effects (font (size 1.27 1.27)) hide)
     )
+    (property "MANUFACTURER" "BL-HG036D-AV-TRB" (id 4) (at 213.106 106.045 0)
+      (effects (font (size 1.27 1.27)) hide)
+    )
     (pin "1")
     (pin "2")
@@
       (effects (font (size 1.27 1.27)) (justify left))
     )
-    (property "Value" "~" (id 1) (at 228.981 153.6699 90)
-      (effects (font (size 1.27 1.27)) (justify left))
-    )
-    (property "Footprint" "" (id 2) (at 223.901 157.48 0)
+    (property "Value" "TestPoint" (id 1) (at 228.981 153.6699 90)
+      (effects (font (size 1.27 1.27)) (justify left))
+    )
+    (property "Footprint" "TestPoint:TestPoint_THTPad_2.0x2.0mm_Drill1.0mm" (id 2) (at 223.901 157.48 0)
       (effects (font (size 1.27 1.27)) hide)
     )
@@
       (effects (font (size 1.27 1.27)) (justify left))
     )
-    (property "Value" "~" (id 1) (at 228.981 151.1299 90)
-      (effects (font (size 1.27 1.27)) (justify left))
-    )
-    (property "Footprint" "" (id 2) (at 223.901 154.94 0)
+    (property "Value" "TestPoint" (id 1) (at 228.981 151.1299 90)
+      (effects (font (size 1.27 1.27)) (justify left))
+    )
+    (property "Footprint" "TestPoint:TestPoint_THTPad_2.0x2.0mm_Drill1.0mm" (id 2) (at 223.901 154.94 0)
       (effects (font (size 1.27 1.27)) hide)
     )
@@
       (effects (font (size 1.27 1.27)) (justify left))
     )
-    (property "Footprint" "" (id 2) (at 223.012 98.679 90)
+    (property "Footprint" "Resistor_SMD:R_0603_1608Metric" (id 2) (at 223.012 98.679 90)
       (effects (font (size 1.27 1.27)) hide)
     )
@@
     )
     (property "Datasheet" "~" (id 3) (at 156.21 122.428 0)
+      (effects (font (size 1.27 1.27)) hide)
+    )
+    (property "MANUFACTURER" "CL10A105KB8NNNC" (id 4) (at 156.21 122.428 0)
       (effects (font (size 1.27 1.27)) hide)
     )
@@
       (effects (font (size 1.27 1.27)) (justify left))
     )
-    (property "Value" "~" (id 1) (at 228.981 148.5899 90)
-      (effects (font (size 1.27 1.27)) (justify left))
-    )
-    (property "Footprint" "" (id 2) (at 223.901 152.4 0)
+    (property "Value" "TestPoint" (id 1) (at 228.981 148.5899 90)
+      (effects (font (size 1.27 1.27)) (justify left))
+    )
+    (property "Footprint" "TestPoint:TestPoint_THTPad_2.0x2.0mm_Drill1.0mm" (id 2) (at 223.901 152.4 0)
       (effects (font (size 1.27 1.27)) hide)
     )
@@
       (effects (font (size 1.27 1.27)) (justify left))
     )
-    (property "Value" "~" (id 1) (at 228.981 146.0499 90)
-      (effects (font (size 1.27 1.27)) (justify left))
-    )
-    (property "Footprint" "" (id 2) (at 223.901 149.86 0)
-      (effects (font (size 1.27 1.27)) hide)
-    )
+    (property "Value" "TestPoint" (id 1) (at 228.981 146.0499 90)
+      (effects (font (size 1.27 1.27)) (justify left))
+    )
+    (property "Footprint" "TestPoint:TestPoint_THTPad_2.0x2.0mm_Drill1.0mm" (id 2) (at 223.901 149.86 0)
+      (effects (font (size 1.27 1.27)) hide)
+    )

Commit message: No clue what changed
Parts:
- added C?: 0.1u, symbol Device:C
- added C?: C, symbol Device:C
Connections:
- net GND: now also C?.2, C?.2
- net VBUS: now also C?.1, C?.1
Changed lines of the file:
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@@
   (junction (at 182.626 127) (diameter 0) (color 0 0 0 0)
   )
+  (junction (at 180.594 32.004) (diameter 0) (color 0 0 0 0)
+  )
   (junction (at 149.606 81.28) (diameter 0) (color 0 0 0 0)
+  )
+  (junction (at 180.594 39.624) (diameter 0) (color 0 0 0 0)
   )
   (junction (at 112.776 105.41) (diameter 0) (color 0 0 0 0)
@@
     (stroke (width 0) (type default) (color 0 0 0 0))
   )
+  (wire (pts (xy 180.594 42.291) (xy 180.594 39.624))
+    (stroke (width 0) (type default) (color 0 0 0 0))
+  )
   (wire (pts (xy 149.606 78.74) (xy 149.606 81.28))
     (stroke (width 0) (type default) (color 0 0 0 0))
@@
     (stroke (width 0) (type default) (color 0 0 0 0))
   )
+  (wire (pts (xy 180.594 39.624) (xy 185.42 39.624))
+    (stroke (width 0) (type default) (color 0 0 0 0))
+  )
   (wire (pts (xy 46.228 99.822) (xy 82.677 99.822))
     (stroke (width 0) (type default) (color 0 0 0 0))
@@
     (stroke (width 0) (type default) (color 0 0 0 0))
   )
+  (wire (pts (xy 175.387 39.624) (xy 180.594 39.624))
+    (stroke (width 0) (type default) (color 0 0 0 0))
+  )
   (wire (pts (xy 164.846 104.14) (xy 156.21 104.14))
     (stroke (width 0) (type default) (color 0 0 0 0))
@@
     (stroke (width 0) (type default) (color 0 0 0 0))
   )
+  (wire (pts (xy 180.594 30.861) (xy 180.594 32.004))
+    (stroke (width 0) (type default) (color 0 0 0 0))
+  )
   (bus (pts (xy 85.217 106.172) (xy 86.487 106.172))
     (stroke (width 0) (type default) (color 0 0 0 0))
   )
+  (wire (pts (xy 180.594 32.004) (xy 185.42 32.004))
+    (stroke (width 0) (type default) (color 0 0 0 0))
+  )
   (wire (pts (xy 182.626 127) (xy 185.166 127))
     (stroke (width 0) (type default) (color 0 0 0 0))
@@
   )
   (wire (pts (xy 120.396 97.79) (xy 133.731 97.79))
+    (stroke (width 0) (type default) (color 0 0 0 0))
+  )
+  (wire (pts (xy 175.387 32.004) (xy 180.594 32.004))
     (stroke (width 0) (type default) (color 0 0 0 0))
   )
@@
     )
     (property "Datasheet" "" (id 3) (at 182.626 128.905 0)
+      (effects (font (size 1.27 1.27)) hide)
+    )
+    (pin "1")
+  )
+  (symbol (lib_id "Device:C") (at 175.387 35.814 0) (unit 1)
+    (in_bom yes) (on_board yes) (fields_autoplaced)
+    (property "Reference" "C?" (id 0) (at 179.07 34.5439 0)
+      (effects (font (size 1.27 1.27)) (justify left))
+    )
+    (property "Value" "0.1u" (id 1) (at 179.07 37.0839 0)
+      (effects (font (size 1.27 1.27)) (justify left))
+    )
+    (property "Footprint" "" (id 2) (at 176.3522 39.624 0)
+      (effects (font (size 1.27 1.27)) hide)
+    )
+    (property "Datasheet" "~" (id 3) (at 175.387 35.814 0)
+      (effects (font (size 1.27 1.27)) hide)
+    )
+    (pin "1")
+    (pin "2")
+  )
+  (symbol (lib_id "power:VBUS") (at 180.594 30.861 0) (unit 1)
+    (in_bom yes) (on_board yes) (fields_autoplaced)
+    (property "Reference" "#PWR?" (id 0) (at 180.594 34.671 0)
+      (effects (font (size 1.27 1.27)) hide)
+    )
+    (property "Value" "VBUS" (id 1) (at 180.594 25.781 0))
+    (property "Footprint" "" (id 2) (at 180.594 30.861 0)
+      (effects (font (size 1.27 1.27)) hide)
+    )
+    (property "Datasheet" "" (id 3) (at 180.594 30.861 0)
       (effects (font (size 1.27 1.27)) hide)
     )
@@
     (pin "1")
   )
+  (symbol (lib_id "Device:C") (at 185.42 35.814 0) (unit 1)
+    (in_bom yes) (on_board yes) (fields_autoplaced)
+    (property "Reference" "C?" (id 0) (at 189.103 34.5439 0)
+      (effects (font (size 1.27 1.27)) (justify left))
+    )
+    (property "Value" "C" (id 1) (at 189.103 37.0839 0)
+      (effects (font (size 1.27 1.27)) (justify left))
+    )
+    (property "Footprint" "" (id 2) (at 186.3852 39.624 0)
+      (effects (font (size 1.27 1.27)) hide)
+    )
+    (property "Datasheet" "~" (id 3) (at 185.42 35.814 0)
+      (effects (font (size 1.27 1.27)) hide)
+    )
+    (pin "1")
+    (pin "2")
+  )
   (symbol (lib_id "Connector:TestPoint") (at 223.901 149.86 270) (unit 1)
     (in_bom yes) (on_board yes)
@@
     (pin "5")
   )
+  (symbol (lib_id "power:GND") (at 180.594 42.291 0) (unit 1)
+    (in_bom yes) (on_board yes) (fields_autoplaced)
+    (property "Reference" "#PWR?" (id 0) (at 180.594 48.641 0)
+      (effects (font (size 1.27 1.27)) hide)
+    )
+    (property "Value" "~" (id 1) (at 180.594 47.117 0))
+    (property "Footprint" "" (id 2) (at 180.594 42.291 0)
+      (effects (font (size 1.27 1.27)) hide)
+    )
+    (property "Datasheet" "" (id 3) (at 180.594 42.291 0)
+      (effects (font (size 1.27 1.27)) hide)
+    )
+    (pin "1")
+  )
   (symbol (lib_id "power:+3V3") (at 69.088 90.932 0) (unit 1)
