File: Electrical/Board Files/Debug.kicad_sch (KiCad schematic)
At the start: 18 parts, among them J2 Conn_01x05_Female, J3 USB_B_Micro, U8 FT231XS

Commit message: Adding footprints
Parts:
- C40: renamed from C36; footprint (none) -> Capacitor_SMD:C_0805_2012Metric
- C41: renamed from C?; footprint (none) -> Capacitor_SMD:C_0805_2012Metric
- C42: renamed from C?; value C -> 0.1u; footprint (none) -> Capacitor_SMD:C_0805_2012Metric
- D19: value LED_Small -> RX_LED
- D20: value - -> TX_LED; footprint Diode_SMD:D_SOD-323 -> LED_SMD:LED_0603_1608Metric
- J2: value Conn_01x05_Female -> DEBUG; footprint (none) -> Connector_PinSocket_2.54mm:PinSocket_1x05_P2.54mm_Vertical; symbol Connector:Conn_01x05_Female -> Connector_Generic:Conn_01x05
- J3: footprint (none) -> Connector_USB:USB_Micro-B_Amphenol_10104110_Horizontal
- renumbered R22 to R26, R23 to R27, R24 to R28, R25 to R29, U8 to U10
Changed lines of the file:
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@@
   (symbol (lib_id "Device:LED_Small") (at 221.996 106.045 90) (unit 1)
     (in_bom yes) (on_board yes) (fields_autoplaced)
-    (property "Reference" "D20" (id 0) (at 223.901 104.7114 90)
+    (property "Reference" "D20" (id 0) (at 224.79 105.9814 90)
       (effects (font (size 1.27 1.27)) (justify right))
     )
-    (property "Value" " - " (id 1) (at 223.901 107.2514 90)
+    (property "Value" "TX_LED" (id 1) (at 223.901 107.2514 90)
       (effects (font (size 1.27 1.27)) (justify right) hide)
     )
-    (property "Footprint" "Diode_SMD:D_SOD-323" (id 2) (at 221.996 106.045 90)
+    (property "Footprint" "LED_SMD:LED_0603_1608Metric" (id 2) (at 221.996 106.045 90)
       (effects (font (size 1.27 1.27)) hide)
     )
@@
   (symbol (lib_id "power:GND") (at 182.626 128.905 0) (unit 1)
     (in_bom yes) (on_board yes) (fields_autoplaced)
-    (property "Reference" "#PWR046" (id 0) (at 182.626 135.255 0)
+    (property "Reference" "#PWR054" (id 0) (at 182.626 135.255 0)
       (effects (font (size 1.27 1.27)) hide)
     )
@@
   (symbol (lib_id "Device:C") (at 175.387 35.814 0) (unit 1)
     (in_bom yes) (on_board yes) (fields_autoplaced)
-    (property "Reference" "C?" (id 0) (at 179.07 34.5439 0)
+    (property "Reference" "C41" (id 0) (at 179.07 34.5439 0)
       (effects (font (size 1.27 1.27)) (justify left))
     )
@@
       (effects (font (size 1.27 1.27)) (justify left))
     )
-    (property "Footprint" "" (id 2) (at 176.3522 39.624 0)
+    (property "Footprint" "Capacitor_SMD:C_0805_2012Metric" (id 2) (at 176.3522 39.624 0)
       (effects (font (size 1.27 1.27)) hide)
     )
@@
   (symbol (lib_id "power:VBUS") (at 180.594 30.861 0) (unit 1)
     (in_bom yes) (on_board yes) (fields_autoplaced)
-    (property "Reference" "#PWR?" (id 0) (at 180.594 34.671 0)
+    (property "Reference" "#PWR052" (id 0) (at 180.594 34.671 0)
       (effects (font (size 1.27 1.27)) hide)
     )
@@
     )
     (property "Value" "TestPoint" (id 1) (at 228.981 143.5099 90)
-      (effects (font (size 1.27 1.27)) (justify left))
+      (effects (font (size 1.27 1.27)) (justify left) hide)
     )
     (property "Footprint" "TestPoint:TestPoint_THTPad_2.0x2.0mm_Drill1.0mm" (id 2) (at 223.901 147.32 0)
@@
   (symbol (lib_id "Device:R_US") (at 213.106 98.425 0) (unit 1)
     (in_bom yes) (on_board yes) (fields_autoplaced)
-    (property "Reference" "R24" (id 0) (at 215.011 97.1549 0)
+    (property "Reference" "R28" (id 0) (at 215.011 97.1549 0)
       (effects (font (size 1.27 1.27)) (justify left))
     )
@@
   (symbol (lib_id "Device:R_Small_US") (at 141.986 93.98 90) (unit 1)
     (in_bom yes) (on_board yes)
-    (property "Reference" "R22" (id 0) (at 141.986 95.885 90))
+    (property "Reference" "R26" (id 0) (at 141.986 95.885 90))
     (property "Value" "27R" (id 1) (at 146.431 92.71 90))
     (property "Footprint" "Resistor_SMD:R_0603_1608Metric" (id 2) (at 141.986 93.98 0)
@@
   (symbol (lib_id "power:VBUS") (at 149.606 78.74 0) (unit 1)
     (in_bom yes) (on_board yes) (fields_autoplaced)
-    (property "Reference" "#PWR045" (id 0) (at 149.606 82.55 0)
+    (property "Reference" "#PWR051" (id 0) (at 149.606 82.55 0)
       (effects (font (size 1.27 1.27)) hide)
     )
@@
   (symbol (lib_id "power:GND") (at 69.088 108.204 0) (unit 1)
     (in_bom yes) (on_board yes) (fields_autoplaced)
-    (property "Reference" "#PWR043" (id 0) (at 69.088 114.554 0)
+    (property "Reference" "#PWR049" (id 0) (at 69.088 114.554 0)
       (effects (font (size 1.27 1.27)) hide)
     )
@@
   (symbol (lib_id "Device:R_Small_US") (at 141.986 99.06 90) (unit 1)
     (in_bom yes) (on_board yes)
-    (property "Reference" "R23" (id 0) (at 142.621 100.965 90))
+    (property "Reference" "R27" (id 0) (at 142.621 100.965 90))
     (property "Value" "27R" (id 1) (at 145.796 97.79 90))
     (property "Footprint" "Resistor_SMD:R_0603_1608Metric" (id 2) (at 141.986 99.06 0)
@@
   (symbol (lib_id "power:GND") (at 110.236 109.22 0) (unit 1)
     (in_bom yes) (on_board yes) (fields_autoplaced)
-    (property "Reference" "#PWR044" (id 0) (at 110.236 115.57 0)
+    (property "Reference" "#PWR050" (id 0) (at 110.236 115.57 0)
       (effects (font (size 1.27 1.27)) hide)
     )
@@
   (symbol (lib_id "Device:LED_Small") (at 213.106 106.045 90) (unit 1)
     (in_bom yes) (on_board yes) (fields_autoplaced)
-    (property "Reference" "D19" (id 0) (at 215.011 104.7114 90)
+    (property "Reference" "D19" (id 0) (at 215.9 105.9814 90)
       (effects (font (size 1.27 1.27)) (justify right))
     )
-    (property "Value" "LED_Small" (id 1) (at 215.011 107.2514 90)
+    (property "Value" "RX_LED" (id 1) (at 215.011 107.2514 90)
       (effects (font (size 1.27 1.27)) (justify right) hide)
     )
@@
     )
     (property "Value" "TestPoint" (id 1) (at 228.981 153.6699 90)
-      (effects (font (size 1.27 1.27)) (justify left))
+      (effects (font (size 1.27 1.27)) (justify left) hide)
     )
     (property "Footprint" "TestPoint:TestPoint_THTPad_2.0x2.0mm_Drill1.0mm" (id 2) (at 223.901 157.48 0)
@@
   (symbol (lib_id "Device:C") (at 185.42 35.814 0) (unit 1)
     (in_bom yes) (on_board yes) (fields_autoplaced)
-    (property "Reference" "C?" (id 0) (at 189.103 34.5439 0)
-      (effects (font (size 1.27 1.27)) (justify left))
-    )
-    (property "Value" "C" (id 1) (at 189.103 37.0839 0)
-      (effects (font (size 1.27 1.27)) (justify left))
-    )
-    (property "Footprint" "" (id 2) (at 186.3852 39.624 0)
+    (property "Reference" "C42" (id 0) (at 189.23 34.5439 0)
+      (effects (font (size 1.27 1.27)) (justify left))
+    )
+    (property "Value" "0.1u" (id 1) (at 189.23 37.0839 0)
+      (effects (font (size 1.27 1.27)) (justify left))
+    )
+    (property "Footprint" "Capacitor_SMD:C_0805_2012Metric" (id 2) (at 186.3852 39.624 0)
       (effects (font (size 1.27 1.27)) hide)
     )
@@
     )
     (property "Value" "TestPoint" (id 1) (at 228.981 151.1299 90)
-      (effects (font (size 1.27 1.27)) (justify left))
+      (effects (font (size 1.27 1.27)) (justify left) hide)
     )
     (property "Footprint" "TestPoint:TestPoint_THTPad_2.0x2.0mm_Drill1.0mm" (id 2) (at 223.901 154.94 0)
@@
   (symbol (lib_id "Device:R_US") (at 221.996 98.425 0) (unit 1)
     (in_bom yes) (on_board yes) (fields_autoplaced)
-    (property "Reference" "R25" (id 0) (at 223.901 97.1549 0)
+    (property "Reference" "R29" (id 0) (at 223.901 97.1549 0)
       (effects (font (size 1.27 1.27)) (justify left))
     )
@@
     (pin "2")
   )
-  (symbol (lib_id "Connector:Conn_01x05_Female") (at 41.148 99.822 0) (mirror y) (unit 1)
-    (in_bom yes) (on_board yes) (fields_autoplaced)
-    (property "Reference" "J2" (id 0) (at 41.783 88.9 0))
-    (property "Value" "Conn_01x05_Female" (id 1) (at 41.783 91.44 0))
-    (property "Footprint" "" (id 2) (at 41.148 99.822 0)
+  (symbol (lib_id "Connector_Generic:Conn_01x05") (at 41.148 99.822 0) (mirror y) (unit 1)
+    (in_bom yes) (on_board yes) (fields_autoplaced)
+    (property "Reference" "J2" (id 0) (at 41.148 90.17 0))
+    (property "Value" "DEBUG" (id 1) (at 41.783 91.44 0)
+      (effects (font (size 1.27 1.27)) hide)
+    )
+    (property "Footprint" "Connector_PinSocket_2.54mm:PinSocket_1x05_P2.54mm_Vertical" (id 2) (at 41.148 99.822 0)
       (effects (font (size 1.27 1.27)) hide)
     )
@@
   (symbol (lib_id "power:GND") (at 180.594 42.291 0) (unit 1)
     (in_bom yes) (on_board yes) (fields_autoplaced)
-    (property "Reference" "#PWR?" (id 0) (at 180.594 48.641 0)
+    (property "Reference" "#PWR053" (id 0) (at 180.594 48.641 0)
       (effects (font (size 1.27 1.27)) hide)
     )
@@
   (symbol (lib_id "power:+3V3") (at 69.088 90.932 0) (unit 1)
     (in_bom yes) (on_board yes) (fields_autoplaced)
-    (property "Reference" "#PWR042" (id 0) (at 69.088 94.742 0)
+    (property "Reference" "#PWR048" (id 0) (at 69.088 94.742 0)
       (effects (font (size 1.27 1.27)) hide)
     )
@@
   (symbol (lib_id "Device:C_Small") (at 156.21 122.428 0) (unit 1)
     (in_bom yes) (on_board yes) (fields_autoplaced)
-    (property "Reference" "C36" (id 0) (at 158.75 121.1642 0)
+    (property "Reference" "C40" (id 0) (at 158.75 121.1642 0)
       (effects (font (size 1.27 1.27)) (justify left))
     )
@@
       (effects (font (size 1.27 1.27)) (justify left))
     )
-    (property "Footprint" "" (id 2) (at 156.21 122.428 0)
+    (property "Footprint" "Capacitor_SMD:C_0805_2012Metric" (id 2) (at 156.21 122.428 0)
       (effects (font (size 1.27 1.27)) hide)
     )
@@
   (symbol (lib_id "Interface_USB:FT231XS") (at 182.626 104.14 0) (unit 1)
     (in_bom yes) (on_board yes) (fields_autoplaced)
-    (property "Reference" "U8" (id 0) (at 187.1854 80.01 0)
+    (property "Reference" "U10" (id 0) (at 187.1854 80.01 0)
       (effects (font (size 1.27 1.27)) (justify left))
     )
@@
     )
     (property "Value" "TestPoint" (id 1) (at 228.981 148.5899 90)
-      (effects (font (size 1.27 1.27)) (justify left))
+      (effects (font (size 1.27 1.27)) (justify left) hide)
     )
     (property "Footprint" "TestPoint:TestPoint_THTPad_2.0x2.0mm_Drill1.0mm" (id 2) (at 223.901 152.4 0)
@@
     )
     (property "Value" "TestPoint" (id 1) (at 228.981 146.0499 90)
-      (effects (font (size 1.27 1.27)) (justify left))
+      (effects (font (size 1.27 1.27)) (justify left) hide)
     )
     (property "Footprint" "TestPoint:TestPoint_THTPad_2.0x2.0mm_Drill1.0mm" (id 2) (at 223.901 149.86 0)
@@
     (property "Reference" "J3" (id 0) (at 112.776 82.55 0))
     (property "Value" "USB_B_Micro" (id 1) (at 112.776 85.09 0))
-    (property "Footprint" "" (id 2) (at 116.586 96.52 0)
-      (effects (font (size 1.27 1.27)) hide)
-    )
+    (property "Footprint" "Connector_USB:USB_Micro-B_Amphenol_10104110_Horizontal" (id 2) (at 116.586 96.52 0)
+      (effects (font (size 1.27 1.27)) hide)
+    )
