File: Electrical/Board Files/Joysticks.kicad_sch (KiCad schematic)
At the start: 14 parts, among them U10 DRV5055A2xLPGxQ1, U5 COM-09032, U6 COM-09032, U9 DRV5055A2xLPGxQ1

Commit message: Adding some device footprints and MPN
Parts:
- C27, C28, C29, C30, C37, C39: MANUFACTURER (none) -> CL10A105KB8NNNC
- C31, C32: footprint (none) -> Capacitor_SMD:C_0603_1608Metric; MANUFACTURER (none) -> CC0603KRX7R9BB104
- C38, C40: footprint (none) -> Capacitor_SMD:C_0603_1608Metric; MANUFACTURER (none) -> 0603B103K500NT
Changed lines of the file:
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@@
+      (effects (font (size 1.27 1.27)) hide)
+    )
+    (property "MANUFACTURER" "CL10A105KB8NNNC" (id 4) (at 123.571 111.633 0)
       (effects (font (size 1.27 1.27)) hide)
     )
@@
       (effects (font (size 1.27 1.27)) hide)
     )
+    (property "MANUFACTURER" "CL10A105KB8NNNC" (id 4) (at 128.27 100.965 0)
+      (effects (font (size 1.27 1.27)) hide)
+    )
     (pin "1")
     (pin "2")
@@
       (effects (font (size 1.27 1.27)) (justify left))
     )
-    (property "Footprint" "" (id 2) (at 153.924 162.814 0)
+    (property "Footprint" "Capacitor_SMD:C_0603_1608Metric" (id 2) (at 153.924 162.814 0)
       (effects (font (size 1.27 1.27)) hide)
     )
@@
       (effects (font (size 1.27 1.27)) hide)
     )
+    (property "MANUFACTURER" "0603B103K500NT" (id 4) (at 153.924 162.814 0)
+      (effects (font (size 1.27 1.27)) hide)
+    )
     (pin "1")
     (pin "2")
@@
     )
     (property "Datasheet" "~" (id 3) (at 144.272 162.814 0)
+      (effects (font (size 1.27 1.27)) hide)
+    )
+    (property "MANUFACTURER" "CL10A105KB8NNNC" (id 4) (at 144.272 162.814 0)
       (effects (font (size 1.27 1.27)) hide)
     )
@@
       (effects (font (size 1.27 1.27)) (justify left))
     )
-    (property "Footprint" "" (id 2) (at 135.763 72.644 0)
+    (property "Footprint" "Capacitor_SMD:C_0603_1608Metric" (id 2) (at 135.763 72.644 0)
       (effects (font (size 1.27 1.27)) hide)
     )
     (property "Datasheet" "~" (id 3) (at 135.763 72.644 0)
+      (effects (font (size 1.27 1.27)) hide)
+    )
+    (property "MANUFACTURER" "CC0603KRX7R9BB104" (id 4) (at 135.763 72.644 0)
       (effects (font (size 1.27 1.27)) hide)
     )
@@
       (effects (font (size 1.27 1.27)) hide)
     )
+    (property "MANUFACTURER" "CL10A105KB8NNNC" (id 4) (at 123.571 83.439 0)
+      (effects (font (size 1.27 1.27)) hide)
+    )
     (pin "1")
     (pin "2")
@@
       (effects (font (size 1.27 1.27)) (justify left))
     )
-    (property "Footprint" "" (id 2) (at 104.394 163.068 0)
+    (property "Footprint" "Capacitor_SMD:C_0603_1608Metric" (id 2) (at 104.394 163.068 0)
       (effects (font (size 1.27 1.27)) hide)
     )
@@
       (effects (font (size 1.27 1.27)) hide)
     )
+    (property "MANUFACTURER" "0603B103K500NT" (id 4) (at 104.394 163.068 0)
+      (effects (font (size 1.27 1.27)) hide)
+    )
     (pin "1")
     (pin "2")
@@
       (effects (font (size 1.27 1.27)) (justify left))
     )
-    (property "Footprint" "" (id 2) (at 135.89 100.965 0)
+    (property "Footprint" "Capacitor_SMD:C_0603_1608Metric" (id 2) (at 135.89 100.965 0)
       (effects (font (size 1.27 1.27)) hide)
     )
@@
       (effects (font (size 1.27 1.27)) hide)
     )
+    (property "MANUFACTURER" "CC0603KRX7R9BB104" (id 4) (at 135.89 100.965 0)
+      (effects (font (size 1.27 1.27)) hide)
+    )
     (pin "1")
     (pin "2")
@@
     )
     (property "Datasheet" "~" (id 3) (at 94.742 163.068 0)
+      (effects (font (size 1.27 1.27)) hide)
+    )
+    (property "MANUFACTURER" "CL10A105KB8NNNC" (id 4) (at 94.742 163.068 0)
       (effects (font (size 1.27 1.27)) hide)
     )
@@
       (effects (font (size 1.27 1.27)) hide)
     )
+    (property "MANUFACTURER" "CL10A105KB8NNNC" (id 4) (at 128.143 72.644 0)
+      (effects (font (size 1.27 1.27)) hide)
+    )

Commit message: Adding footprints
Parts:
- C27: renamed from C37; footprint (none) -> Capacitor_SMD:C_0805_2012Metric
- C28: renamed from C38; footprint Capacitor_SMD:C_0603_1608Metric -> Capacitor_SMD:C_0805_2012Metric
- C29: renamed from C27; footprint (none) -> Capacitor_SMD:C_0805_2012Metric
- C30: renamed from C28; footprint (none) -> Capacitor_SMD:C_0805_2012Metric
- C31: renamed from C29; footprint (none) -> Capacitor_SMD:C_0805_2012Metric
- C32: renamed from C30; footprint (none) -> Capacitor_SMD:C_0805_2012Metric
- C33: renamed from C31; footprint Capacitor_SMD:C_0603_1608Metric -> Capacitor_SMD:C_0805_2012Metric
- C34: renamed from C32; footprint Capacitor_SMD:C_0603_1608Metric -> Capacitor_SMD:C_0805_2012Metric
- C35: renamed from C39; footprint (none) -> Capacitor_SMD:C_0805_2012Metric
- C36: renamed from C40; footprint Capacitor_SMD:C_0603_1608Metric -> Capacitor_SMD:C_0805_2012Metric
- U7: renamed from U5; footprint (none) -> COM-09032:XDCR_COM-09032
- U8: renamed from U6; footprint (none) -> COM-09032:XDCR_COM-09032
- renumbered U9 to U5, U10 to U6
