File: Electrical/Board Files/ScanMatrix.kicad_sch (KiCad schematic)
At the start: 33 parts

Commit message: Adding new block diagram
Parts:
- U? (x3): value (none) -> 74LVC3G17
Changed lines of the file:
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@@
     (in_bom yes) (on_board yes) (fields_autoplaced)
     (property "Reference" "U?" (id 0) (at 201.295 76.962 0))
-    (property "Value" "" (id 1) (at 201.295 79.502 0))
+    (property "Value" "74LVC3G17" (id 1) (at 201.295 79.502 0))
     (property "Footprint" "" (id 2) (at 201.93 84.836 0)
       (effects (font (size 1.27 1.27)) hide)
@@
     (in_bom yes) (on_board yes) (fields_autoplaced)
     (property "Reference" "U?" (id 0) (at 201.041 60.452 0))
-    (property "Value" "" (id 1) (at 201.041 62.992 0))
+    (property "Value" "74LVC3G17" (id 1) (at 201.041 62.992 0))
     (property "Footprint" "" (id 2) (at 201.676 68.326 0)
       (effects (font (size 1.27 1.27)) hide)
@@
       (effects (font (size 1.27 1.27)) hide)
     )
-    (property "Value" "" (id 1) (at 223.901 92.964 0))
+    (property "Value" "GND" (id 1) (at 223.901 92.964 0))
     (property "Footprint" "" (id 2) (at 223.901 87.376 0)
       (effects (font (size 1.27 1.27)) hide)
@@
     (in_bom yes) (on_board yes) (fields_autoplaced)
     (property "Reference" "U?" (id 0) (at 200.533 45.212 0))
-    (property "Value" "" (id 1) (at 200.533 47.752 0))
+    (property "Value" "74LVC3G17" (id 1) (at 200.533 47.752 0))
     (property "Footprint" "" (id 2) (at 201.168 53.594 0)
       (effects (font (size 1.27 1.27)) hide)

Commit message: Updating for 3v3 operation
Connections:
- net +3V0 renamed +3V3
Changed lines of the file:
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@@
     (effects (font (size 1.27 1.27)) (justify right))
   )
-  (hierarchical_label "COL[1..2]" (shape input) (at 46.99 34.544 180)
+  (hierarchical_label "COL[1..2]" (shape output) (at 46.99 34.544 180)
     (effects (font (size 1.27 1.27)) (justify right))
   )
@@
     (pin "1")
     (pin "2")
-  )
-  (symbol (lib_id "power:+3V0") (at 223.901 80.264 0) (unit 1)
-    (in_bom yes) (on_board yes) (fields_autoplaced)
-    (property "Reference" "#PWR?" (id 0) (at 223.901 84.074 0)
-      (effects (font (size 1.27 1.27)) hide)
-    )
-    (property "Value" "+3V0" (id 1) (at 223.901 74.803 0))
-    (property "Footprint" "" (id 2) (at 223.901 80.264 0)
-      (effects (font (size 1.27 1.27)) hide)
-    )
-    (property "Datasheet" "" (id 3) (at 223.901 80.264 0)
-      (effects (font (size 1.27 1.27)) hide)
-    )
-    (pin "1")
   )
   (symbol (lib_id "Device:D_Small") (at 122.428 129.032 180) (unit 1)
@@
     (pin "2")
   )
+  (symbol (lib_id "power:+3V3") (at 223.901 80.264 0) (unit 1)
+    (in_bom yes) (on_board yes) (fields_autoplaced)
+    (property "Reference" "#PWR?" (id 0) (at 223.901 84.074 0)
+      (effects (font (size 1.27 1.27)) hide)
+    )
+    (property "Value" "+3V3" (id 1) (at 223.901 74.93 0))
+    (property "Footprint" "" (id 2) (at 223.901 80.264 0)
+      (effects (font (size 1.27 1.27)) hide)
+    )
+    (property "Datasheet" "" (id 3) (at 223.901 80.264 0)
+      (effects (font (size 1.27 1.27)) hide)
+    )
+    (pin "1")
+  )
   (symbol (lib_id "74xGxx:74LVC3G17") (at 201.168 53.594 0) (unit 1)

Commit message: Added Xbee libs and bus aliases
Parts:
- gave numbers to parts that had none: 11
Other:
- title: (none) -> Robotics Controller
Changed lines of the file:
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@@
 (kicad_sch (version 20211123) (generator eeschema)
   (paper "A4")
+  (title_block
+    (title "Robotics Controller")
+    (rev "A")
+  )
   (junction (at 104.648 121.412) (diameter 0) (color 0 0 0 0)
   )
@@
   (symbol (lib_id "Switch:SW_DIP_x01") (at 112.268 174.752 0) (unit 1)
     (in_bom yes) (on_board yes)
-    (property "Reference" "SW?" (id 0) (at 112.268 170.942 0))
+    (property "Reference" "SW13" (id 0) (at 112.268 170.942 0))
     (property "Value" "~" (id 1) (at 112.268 169.672 0))
     (property "Footprint" "" (id 2) (at 112.268 174.752 0)
@@
   (symbol (lib_id "74xGxx:74LVC3G17") (at 201.93 84.836 0) (unit 3)
     (in_bom yes) (on_board yes) (fields_autoplaced)
-    (property "Reference" "U?" (id 0) (at 201.295 76.962 0))
+    (property "Reference" "U4" (id 0) (at 201.295 76.962 0))
     (property "Value" "74LVC3G17" (id 1) (at 201.295 79.502 0))
     (property "Footprint" "" (id 2) (at 201.93 84.836 0)
@@
   (symbol (lib_id "74xGxx:74LVC3G17") (at 201.676 68.326 0) (unit 2)
     (in_bom yes) (on_board yes) (fields_autoplaced)
-    (property "Reference" "U?" (id 0) (at 201.041 60.452 0))
+    (property "Reference" "U4" (id 0) (at 201.041 60.452 0))
     (property "Value" "74LVC3G17" (id 1) (at 201.041 62.992 0))
     (property "Footprint" "" (id 2) (at 201.676 68.326 0)
@@
   (symbol (lib_id "Device:D_Small") (at 122.428 158.242 180) (unit 1)
     (in_bom yes) (on_board yes)
-    (property "Reference" "D?" (id 0) (at 122.428 155.702 0))
+    (property "Reference" "D13" (id 0) (at 122.428 155.702 0))
     (property "Value" "~" (id 1) (at 122.428 154.432 0))
     (property "Footprint" "" (id 2) (at 122.428 158.242 90)
@@
   (symbol (lib_id "Switch:SW_DIP_x01") (at 154.178 158.242 0) (unit 1)
     (in_bom yes) (on_board yes)
-    (property "Reference" "SW?" (id 0) (at 154.178 154.432 0))
+    (property "Reference" "SW14" (id 0) (at 154.178 154.432 0))
     (property "Value" "~" (id 1) (at 154.178 153.162 0))
     (property "Footprint" "" (id 2) (at 154.178 158.242 0)
@@
   (symbol (lib_id "power:GND") (at 223.901 87.376 0) (unit 1)
     (in_bom yes) (on_board yes) (fields_autoplaced)
-    (property "Reference" "#PWR?" (id 0) (at 223.901 93.726 0)
+    (property "Reference" "#PWR019" (id 0) (at 223.901 93.726 0)
       (effects (font (size 1.27 1.27)) hide)
     )
@@
   (symbol (lib_id "Device:D_Small") (at 122.428 174.752 180) (unit 1)
     (in_bom yes) (on_board yes)
-    (property "Reference" "D?" (id 0) (at 122.428 172.212 0))
+    (property "Reference" "D14" (id 0) (at 122.428 172.212 0))
     (property "Value" "~" (id 1) (at 122.428 170.942 0))
     (property "Footprint" "" (id 2) (at 122.428 174.752 90)
@@
   (symbol (lib_id "Device:C_Small") (at 216.281 84.836 0) (unit 1)
     (in_bom yes) (on_board yes)
-    (property "Reference" "C?" (id 0) (at 212.344 83.566 0)
+    (property "Reference" "C25" (id 0) (at 212.344 83.566 0)
       (effects (font (size 1.27 1.27)) (justify left))
     )
@@
   (symbol (lib_id "Device:D_Small") (at 164.338 158.242 180) (unit 1)
     (in_bom yes) (on_board yes)
-    (property "Reference" "D?" (id 0) (at 164.338 155.702 0))
+    (property "Reference" "D15" (id 0) (at 164.338 155.702 0))
     (property "Value" "~" (id 1) (at 164.338 154.432 0))
     (property "Footprint" "" (id 2) (at 164.338 158.242 90)
@@
   (symbol (lib_id "Device:D_Small") (at 164.338 174.752 180) (unit 1)
     (in_bom yes) (on_board yes)
-    (property "Reference" "D?" (id 0) (at 164.338 172.212 0))
+    (property "Reference" "D16" (id 0) (at 164.338 172.212 0))
     (property "Value" "~" (id 1) (at 164.338 170.942 0))
     (property "Footprint" "" (id 2) (at 164.338 174.752 90)
@@
   (symbol (lib_id "Device:C_Small") (at 223.901 84.836 0) (unit 1)
     (in_bom yes) (on_board yes)
-    (property "Reference" "C?" (id 0) (at 226.441 83.566 0)
+    (property "Reference" "C26" (id 0) (at 226.441 83.566 0)
       (effects (font (size 1.27 1.27)) (justify left))
     )
@@
   (symbol (lib_id "Switch:SW_DIP_x01") (at 112.268 158.242 0) (unit 1)
     (in_bom yes) (on_board yes)
-    (property "Reference" "SW?" (id 0) (at 112.268 154.432 0))
+    (property "Reference" "SW12" (id 0) (at 112.268 154.432 0))
     (property "Value" "~" (id 1) (at 112.268 153.162 0))
     (property "Footprint" "" (id 2) (at 112.268 158.242 0)
@@
   (symbol (lib_id "Switch:SW_DIP_x01") (at 154.178 174.752 0) (unit 1)
     (in_bom yes) (on_board yes)
-    (property "Reference" "SW?" (id 0) (at 154.178 170.942 0))
+    (property "Reference" "SW15" (id 0) (at 154.178 170.942 0))
     (property "Value" "~" (id 1) (at 154.178 169.672 0))
     (property "Footprint" "" (id 2) (at 154.178 174.752 0)
@@
   (symbol (lib_id "power:+3V3") (at 223.901 80.264 0) (unit 1)
     (in_bom yes) (on_board yes) (fields_autoplaced)
-    (property "Reference" "#PWR?" (id 0) (at 223.901 84.074 0)
+    (property "Reference" "#PWR018" (id 0) (at 223.901 84.074 0)
       (effects (font (size 1.27 1.27)) hide)
     )
@@
   (symbol (lib_id "74xGxx:74LVC3G17") (at 201.168 53.594 0) (unit 1)
     (in_bom yes) (on_board yes) (fields_autoplaced)
-    (property "Reference" "U?" (id 0) (at 200.533 45.212 0))
+    (property "Reference" "U4" (id 0) (at 200.533 45.212 0))
     (property "Value" "74LVC3G17" (id 1) (at 200.533 47.752 0))
     (property "Footprint" "" (id 2) (at 201.168 53.594 0)

Commit message: Updating title block fields and adding pdf schematic
Other:
- company: (none) -> Rockerbotics
Changed lines of the file:
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@@
   (title_block
     (title "Robotics Controller")
+    (date "2022-09-02")
     (rev "A")
+    (company "Rockerbotics")
   )
   (junction (at 104.648 121.412) (diameter 0) (color 0 0 0 0)

Commit message: Adding some device footprints and MPN
Parts:
- C25: MANUFACTURER (none) -> CL10A105KB8NNNC
- C26: footprint (none) -> Capacitor_SMD:C_0603_1608Metric; MANUFACTURER (none) -> CC0603KRX7R9BB104
- D1, D10, D13, D14, D15, D16, D2, D3, D4, D5, D6, D7, D8, D9: value ~ -> -; footprint (none) -> Diode_SMD:D_SOD-323; MANUFACTURER (none) -> 1N4148WS
- U4: footprint (none) -> Package_SO:TSSOP-8_3x3mm_P0.65mm

Commit message: No clue what changed
Parts:
- added R? (x4): 10k, symbol Device:R_Small_US
Connections:
- net GND: now also R?.2, R?.2, R?.2, R?.2
- net at D10.1 (K), D15.1 (K), D16.1 (K)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: now also R?.1
- net at D1.1 (K), D13.1 (K), D14.1 (K)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: now also R?.1
- net at U4.3: now also R?.1
- net at U4.5: now also R?.1
- no-connect marks 2 -> 0
Changed lines of the file:
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@@
   (junction (at 166.878 103.632) (diameter 0) (color 0 0 0 0)
   )
+  (junction (at 180.213 68.326) (diameter 0) (color 0 0 0 0)
+  )
   (junction (at 104.648 108.712) (diameter 0) (color 0 0 0 0)
   )
@@
   (junction (at 104.648 150.622) (diameter 0) (color 0 0 0 0)
   )
+  (junction (at 180.213 53.594) (diameter 0) (color 0 0 0 0)
+  )
   (junction (at 124.968 129.032) (diameter 0) (color 0 0 0 0)
   )
   (junction (at 166.878 141.732) (diameter 0) (color 0 0 0 0)
   )
+  (junction (at 200.787 95.631) (diameter 0) (color 0 0 0 0)
+  )
   (junction (at 124.968 103.632) (diameter 0) (color 0 0 0 0)
   )
@@
   (junction (at 223.901 82.296) (diameter 0) (color 0 0 0 0)
   )
-  (no_connect (at 208.28 84.836))
-  (no_connect (at 194.31 84.836))
   (bus_entry (at 225.552 34.544) (size 2.54 2.54)
     (stroke (width 0) (type default) (color 0 0 0 0))
@@
     (stroke (width 0) (type default) (color 0 0 0 0))
   )
+  (wire (pts (xy 194.31 84.836) (xy 194.31 89.408))
+    (stroke (width 0) (type default) (color 0 0 0 0))
+  )
   (bus (pts (xy 94.488 148.082) (xy 94.488 164.592))
     (stroke (width 0) (type default) (color 0 0 0 0))
@@
     (stroke (width 0) (type default) (color 0 0 0 0))
   )
+  (wire (pts (xy 180.213 55.118) (xy 180.213 53.594))
+    (stroke (width 0) (type default) (color 0 0 0 0))
+  )
   (wire (pts (xy 146.558 116.332) (xy 146.558 108.712))
     (stroke (width 0) (type default) (color 0 0 0 0))
@@
     (stroke (width 0) (type default) (color 0 0 0 0))
   )
+  (wire (pts (xy 194.31 94.488) (xy 194.31 95.631))
+    (stroke (width 0) (type default) (color 0 0 0 0))
+  )
+  (wire (pts (xy 180.213 68.326) (xy 194.056 68.326))
+    (stroke (width 0) (type default) (color 0 0 0 0))
+  )
   (wire (pts (xy 104.648 83.312) (xy 97.028 83.312))
     (stroke (width 0) (type default) (color 0 0 0 0))
@@
     (stroke (width 0) (type default) (color 0 0 0 0))
   )
+  (wire (pts (xy 180.213 69.977) (xy 180.213 68.326))
+    (stroke (width 0) (type default) (color 0 0 0 0))
+  )
   (wire (pts (xy 223.901 80.264) (xy 223.901 82.296))
     (stroke (width 0) (type default) (color 0 0 0 0))
@@
     (stroke (width 0) (type default) (color 0 0 0 0))
   )
+  (wire (pts (xy 208.407 84.836) (xy 208.28 84.836))
+    (stroke (width 0) (type default) (color 0 0 0 0))
+  )
   (wire (pts (xy 97.028 150.622) (xy 104.648 150.622))
     (stroke (width 0) (type default) (color 0 0 0 0))
@@
     (stroke (width 0) (type default) (color 0 0 0 0))
   )
+  (wire (pts (xy 180.213 53.594) (xy 193.548 53.594))
+    (stroke (width 0) (type default) (color 0 0 0 0))
+  )
   (wire (pts (xy 104.648 121.412) (xy 104.648 129.032))
     (stroke (width 0) (type default) (color 0 0 0 0))
   )
+  (wire (pts (xy 208.407 95.631) (xy 208.407 94.869))
+    (stroke (width 0) (type default) (color 0 0 0 0))
+  )
   (wire (pts (xy 146.558 83.312) (xy 146.558 90.932))
     (stroke (width 0) (type default) (color 0 0 0 0))
@@
     (stroke (width 0) (type default) (color 0 0 0 0))
   )
+  (wire (pts (xy 194.31 95.631) (xy 200.787 95.631))
+    (stroke (width 0) (type default) (color 0 0 0 0))
+  )
   (wire (pts (xy 146.558 134.112) (xy 104.648 134.112))
     (stroke (width 0) (type default) (color 0 0 0 0))
@@
     (stroke (width 0) (type default) (color 0 0 0 0))
   )
+  (wire (pts (xy 200.787 95.631) (xy 208.407 95.631))
+    (stroke (width 0) (type default) (color 0 0 0 0))
+  )
   (wire (pts (xy 146.558 96.012) (xy 146.558 103.632))
     (stroke (width 0) (type default) (color 0 0 0 0))
   )
-  (wire (pts (xy 124.968 53.594) (xy 193.548 53.594))
+  (wire (pts (xy 124.968 53.594) (xy 180.213 53.594))
+    (stroke (width 0) (type default) (color 0 0 0 0))
+  )
+  (wire (pts (xy 208.407 89.789) (xy 208.407 84.836))
     (stroke (width 0) (type default) (color 0 0 0 0))
   )
@@
     (stroke (width 0) (type default) (color 0 0 0 0))
   )
-  (wire (pts (xy 166.878 68.326) (xy 194.056 68.326))
+  (wire (pts (xy 166.878 68.326) (xy 180.213 68.326))
     (stroke (width 0) (type default) (color 0 0 0 0))
   )
@@
     (pin "2")
   )
+  (symbol (lib_id "Device:R_Small_US") (at 180.213 57.658 0) (unit 1)
+    (in_bom yes) (on_board yes) (fields_autoplaced)
+    (property "Reference" "R?" (id 0) (at 182.626 56.3879 0)
+      (effects (font (size 1.27 1.27)) (justify left))
+    )
+    (property "Value" "10k" (id 1) (at 182.626 58.9279 0)
+      (effects (font (size 1.27 1.27)) (justify left))
+    )
+    (property "Footprint" "" (id 2) (at 180.213 57.658 0)
+      (effects (font (size 1.27 1.27)) hide)
+    )
+    (property "Datasheet" "~" (id 3) (at 180.213 57.658 0)
+      (effects (font (size 1.27 1.27)) hide)
+    )
+    (pin "1")
+    (pin "2")
+  )
   (symbol (lib_id "Switch:SW_DIP_x01") (at 112.268 174.752 0) (unit 1)
     (in_bom yes) (on_board yes)
@@
     (pin "2")
   )
+  (symbol (lib_id "Device:R_Small_US") (at 208.407 92.329 0) (unit 1)
+    (in_bom yes) (on_board yes) (fields_autoplaced)
+    (property "Reference" "R?" (id 0) (at 210.82 91.0589 0)
+      (effects (font (size 1.27 1.27)) (justify left))
+    )
+    (property "Value" "10k" (id 1) (at 210.82 93.5989 0)
+      (effects (font (size 1.27 1.27)) (justify left))
+    )
+    (property "Footprint" "" (id 2) (at 208.407 92.329 0)
+      (effects (font (size 1.27 1.27)) hide)
+    )
+    (property "Datasheet" "~" (id 3) (at 208.407 92.329 0)
+      (effects (font (size 1.27 1.27)) hide)
+    )
+    (pin "1")
+    (pin "2")
+  )
+  (symbol (lib_id "power:GND") (at 180.213 60.198 0) (unit 1)
+    (in_bom yes) (on_board yes) (fields_autoplaced)
+    (property "Reference" "#PWR?" (id 0) (at 180.213 66.548 0)
+      (effects (font (size 1.27 1.27)) hide)
+    )
+    (property "Value" "GND" (id 1) (at 180.213 65.786 0))
+    (property "Footprint" "" (id 2) (at 180.213 60.198 0)
+      (effects (font (size 1.27 1.27)) hide)
+    )
+    (property "Datasheet" "" (id 3) (at 180.213 60.198 0)
+      (effects (font (size 1.27 1.27)) hide)
+    )
+    (pin "1")
+  )
   (symbol (lib_id "Device:D_Small") (at 164.338 141.732 180) (unit 1)
     (in_bom yes) (on_board yes)
@@
     (pin "2")
   )
+  (symbol (lib_id "Device:R_Small_US") (at 180.213 72.517 0) (unit 1)
+    (in_bom yes) (on_board yes) (fields_autoplaced)
+    (property "Reference" "R?" (id 0) (at 182.626 71.2469 0)
+      (effects (font (size 1.27 1.27)) (justify left))
+    )
+    (property "Value" "10k" (id 1) (at 182.626 73.7869 0)
+      (effects (font (size 1.27 1.27)) (justify left))
+    )
+    (property "Footprint" "" (id 2) (at 180.213 72.517 0)
+      (effects (font (size 1.27 1.27)) hide)
+    )
+    (property "Datasheet" "~" (id 3) (at 180.213 72.517 0)
+      (effects (font (size 1.27 1.27)) hide)
+    )
+    (pin "1")
+    (pin "2")
+  )
   (symbol (lib_id "Device:C_Small") (at 216.281 84.836 0) (unit 1)
     (in_bom yes) (on_board yes)
@@
     (pin "2")
   )
+  (symbol (lib_id "power:GND") (at 180.213 75.057 0) (unit 1)
+    (in_bom yes) (on_board yes) (fields_autoplaced)
+    (property "Reference" "#PWR?" (id 0) (at 180.213 81.407 0)
+      (effects (font (size 1.27 1.27)) hide)
+    )
+    (property "Value" "GND" (id 1) (at 180.213 80.645 0))
+    (property "Footprint" "" (id 2) (at 180.213 75.057 0)
+      (effects (font (size 1.27 1.27)) hide)
+    )
+    (property "Datasheet" "" (id 3) (at 180.213 75.057 0)
+      (effects (font (size 1.27 1.27)) hide)
+    )
+    (pin "1")
+  )
   (symbol (lib_id "Device:D_Small") (at 122.428 103.632 180) (unit 1)
     (in_bom yes) (on_board yes)
@@
     (pin "2")
   )
+  (symbol (lib_id "Device:R_Small_US") (at 194.31 91.948 0) (unit 1)
+    (in_bom yes) (on_board yes) (fields_autoplaced)
+    (property "Reference" "R?" (id 0) (at 196.723 90.6779 0)
+      (effects (font (size 1.27 1.27)) (justify left))
+    )
+    (property "Value" "10k" (id 1) (at 196.723 93.2179 0)
+      (effects (font (size 1.27 1.27)) (justify left))
+    )
+    (property "Footprint" "" (id 2) (at 194.31 91.948 0)
+      (effects (font (size 1.27 1.27)) hide)
+    )
+    (property "Datasheet" "~" (id 3) (at 194.31 91.948 0)
+      (effects (font (size 1.27 1.27)) hide)
+    )
+    (pin "1")
+    (pin "2")
+  )
   (symbol (lib_id "Switch:SW_DIP_x01") (at 154.178 174.752 0) (unit 1)
     (in_bom yes) (on_board yes)
@@
     (pin "2")
   )
+  (symbol (lib_id "power:GND") (at 200.787 95.631 0) (unit 1)
+    (in_bom yes) (on_board yes) (fields_autoplaced)
+    (property "Reference" "#PWR?" (id 0) (at 200.787 101.981 0)
+      (effects (font (size 1.27 1.27)) hide)
+    )
+    (property "Value" "GND" (id 1) (at 200.787 101.219 0))
+    (property "Footprint" "" (id 2) (at 200.787 95.631 0)
+      (effects (font (size 1.27 1.27)) hide)
+    )
+    (property "Datasheet" "" (id 3) (at 200.787 95.631 0)
+      (effects (font (size 1.27 1.27)) hide)
+    )
+    (pin "1")
+  )
   (symbol (lib_id "Device:D_Small") (at 122.428 116.332 180) (unit 1)

Commit message: Adding footprints
Parts:
- removed D1, D10, D13, D14, D15, D16, D2, D3, D4, D5, D6, D7, D8, D9: -, Diode_SMD:D_SOD-323, symbol Device:D_Small
- added D10, D11, D12, D13, D14, D15, D16, D3, D4, D5, D6, D7, D8, D9: BAT54J, Diode_SMD:D_SOD-323F, symbol Diode:BAT54J
- C25: footprint (none) -> Capacitor_SMD:C_0805_2012Metric
- C26: footprint Capacitor_SMD:C_0603_1608Metric -> Capacitor_SMD:C_0805_2012Metric
- R11, R12, R13, R14: renamed from R?; footprint (none) -> Resistor_SMD:R_0805_2012Metric
- SW10: renamed from SW7; footprint (none) -> Button_Switch_THT:SW_PUSH-12mm
- SW11: renamed from SW8; footprint (none) -> Button_Switch_THT:SW_PUSH-12mm
- SW12: renamed from SW9; footprint (none) -> Button_Switch_THT:SW_PUSH-12mm
- SW13: renamed from SW10; footprint (none) -> Button_Switch_THT:SW_PUSH-12mm
- SW14, SW15: footprint (none) -> Button_Switch_THT:SW_PUSH-12mm
- SW2: renamed from SW1; footprint (none) -> Button_Switch_THT:SW_PUSH-12mm
- SW3: renamed from SW2; footprint (none) -> Button_Switch_THT:SW_PUSH-12mm
- SW4: renamed from SW3; footprint (none) -> Button_Switch_THT:SW_PUSH-12mm
- SW5: renamed from SW4; footprint (none) -> Button_Switch_THT:SW_PUSH-12mm
- SW6: renamed from SW5; footprint (none) -> Button_Switch_THT:SW_PUSH-12mm
- SW7: renamed from SW12; footprint (none) -> Button_Switch_THT:SW_PUSH-12mm
- SW8: renamed from SW13; footprint (none) -> Button_Switch_THT:SW_PUSH-12mm
- SW9: renamed from SW6; footprint (none) -> Button_Switch_THT:SW_PUSH-12mm
Connections:
- net at SW5.2: now also D6.2 (A)
- net at R11.1, U4.1: now also D3.1 (K), D4.1 (K), D5.1 (K), D6.1 (K), D7.1 (K), D8.1 (K), D9.1 (K)
- net at SW8.2: now also D9.2 (A)
- net at R12.1, U4.6: now also D10.1 (K), D11.1 (K), D12.1 (K), D13.1 (K), D14.1 (K), D15.1 (K), D16.1 (K)
- net at SW10.2: now also D11.2 (A)
- net at SW13.2: now also D14.2 (A)
- net at SW2.2: now also D3.2 (A)
- net at SW7.2: now also D8.2 (A)
- net at SW14.2: now also D15.2 (A)
- net at SW9.2: now also D10.2 (A)
- net at SW6.2: now also D7.2 (A)
- net at SW11.2: now also D12.2 (A)
- net at SW12.2: now also D13.2 (A)
- net at SW15.2: now also D16.2 (A)
- net at SW3.2: now also D4.2 (A)
- net at SW4.2: now also D5.2 (A)
